File: KiCad/SilosProject/List02.kicad_sch (KiCad schematic)
At the start: 122 parts, among them J2 PORT01, J3 PORT03, J4 PORT02, J5 PORT05, J6 PORT04, U10 EL817, U11 EL817, U12 EL817, U13 EL817, U14 EL817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

Commit message: Experement input E2
Connections:
- net GND: now also D33.2 (A), R18.2, U8.2
Changed lines of the file:
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@@
     (pin "4")
+  )
+  (symbol (lib_id "power:GND") (at 104.14 49.53 0) (unit 1)
+    (in_bom yes) (on_board yes) (fields_autoplaced)
+    (property "Reference" "#PWR?" (id 0) (at 104.14 55.88 0)
+      (effects (font (size 1.27 1.27)) hide)
+    )
+    (property "Value" "GND" (id 1) (at 104.14 54.61 0))
+    (property "Footprint" "" (id 2) (at 104.14 49.53 0)
+      (effects (font (size 1.27 1.27)) hide)
+    )
+    (property "Datasheet" "" (id 3) (at 104.14 49.53 0)
+      (effects (font (size 1.27 1.27)) hide)
+    )
+    (pin "1")
   )
   (symbol (lib_id "Isolator:EL817") (at 78.74 40.64 0) (mirror y) (unit 1)
